File: Central Command.sch (KiCad schematic (older format))
At the start: 0 parts

Commit message: Finished assigning pins to the 3 banks of the symbol
Parts:
- added U? (x3): STM32F030C8, symbol STM32F030C8
Changed lines of the file:
@@
 LIBS:contrib
 LIBS:valves
+LIBS:stm32f030c8
+LIBS:Central Command-cache
 EELAYER 25 0
 EELAYER END
@@
 Comment4 ""
 $EndDescr
+$Comp
+L STM32F030C8 U?
+U 1 1 561CB096
+P 4000 1950
+F 0 "U?" H 4500 1550 60  0000 C CNN
+F 1 "STM32F030C8" H 4300 1650 60  0000 C CNN
+F 2 "" H 4000 1950 60  0000 C CNN
+F 3 "" H 4000 1950 60  0000 C CNN
+	1    4000 1950
+	1    0    0    -1
+$EndComp
+$Comp
+L STM32F030C8 U?
+U 2 1 561CB127
+P 4050 4550
+F 0 "U?" H 4550 4150 60  0000 C CNN
+F 1 "STM32F030C8" H 4350 4250 60  0000 C CNN
+F 2 "" H 4050 4550 60  0000 C CNN
+F 3 "" H 4050 4550 60  0000 C CNN
+	2    4050 4550
+	1    0    0    -1
+$EndComp
+$Comp
+L STM32F030C8 U?
+U 3 1 561CB171
+P 7050 2050
+F 0 "U?" H 7550 1650 60  0000 C CNN
+F 1 "STM32F030C8" H 7350 1750 60  0000 C CNN
+F 2 "" H 7050 2050 60  0000 C CNN
+F 3 "" H 7050 2050 60  0000 C CNN
+	3    7050 2050
+	1    0    0    -1
+$EndComp
 $EndSCHEMATC
