File: Central Command.sch (KiCad schematic (older format))
At the start: 12 parts, among them U1 STM32F030C8, Y1 Crystal

Commit message: Associated footprints, created footprints for 2mm connector and did prelim placement
Parts:
- P101, P102: renamed from P?; footprint (none) -> Pin_Headers:Pin_Header_Straight_1x10
- P103, P105: renamed from P?; footprint (none) -> Pin_Headers:Pin_Header_Straight_1x04
- P104, P106: renamed from P?; footprint (none) -> Pin_Headers:Pin_Header_Straight_1x02
- renumbered C2 to C101, C4 to C102, C5 to C103, L1 to L101, U1 to U101, Y1 to Y101
Other:
- note added: "GPIO HEADER 2"
- note removed: "TODO: Get crystal/oscillator"
Changed lines of the file:
@@
 $EndDescr
 $Comp
-L INDUCTOR L1
+L INDUCTOR L101
 U 1 1 5626F24B
 P 4400 700
-F 0 "L1" V 4350 700 50  0000 C CNN
+F 0 "L101" V 4350 700 50  0000 C CNN
 F 1 "INDUCTOR" V 4500 700 50  0000 C CNN
 F 2 "Inductors_NEOSID:Neosid_Inductor_SM1206" H 4400 700 60  0001 C CNN
@@
 $EndComp
 $Comp
-L C C2
+L C C101
 U 1 1 5626F380
 P 5150 850
-F 0 "C2" H 5175 950 50  0000 L CNN
+F 0 "C101" H 5175 950 50  0000 L CNN
 F 1 "C" H 5175 750 50  0000 L CNN
 F 2 "Capacitors_SMD:C_0805" H 5188 700 30  0001 C CNN
@@
 $EndComp
 $Comp
-L GND #PWR02
+L GND #PWR01
 U 1 1 5627066D
 P 3950 3200
-F 0 "#PWR02" H 3950 2950 50  0001 C CNN
+F 0 "#PWR01" H 3950 2950 50  0001 C CNN
 F 1 "GND" H 3950 3050 50  0000 C CNN
 F 2 "" H 3950 3200 60  0000 C CNN
@@
 PA2/PA3 will not have serial for the -C6 chip
 $Comp
-L STM32F030C8 U1
+L STM32F030C8 U101
 U 1 1 564E875E
 P 4200 4500
-F 0 "U1" H 4750 3550 60  0000 C CNN
+F 0 "U101" H 4750 3550 60  0000 C CNN
 F 1 "STM32F030C8" H 4550 5400 60  0000 C CNN
 F 2 "Housings_QFP:LQFP-48_7x7mm_Pitch0.5mm" H 4200 4500 60  0001 C CNN
@@
 $EndComp
 $Comp
-L STM32F030C8 U1
+L STM32F030C8 U101
 U 2 1 564E8A03
 P 4200 6550
-F 0 "U1" H 4750 5600 60  0000 C CNN
+F 0 "U101" H 4750 5600 60  0000 C CNN
 F 1 "STM32F030C8" H 4550 7450 60  0000 C CNN
 F 2 "Housings_QFP:LQFP-48_7x7mm_Pitch0.5mm" H 4200 6550 60  0001 C CNN
@@
 $EndComp
 $Comp
-L STM32F030C8 U1
+L STM32F030C8 U101
 U 3 1 564E8FF6
 P 4200 1950
-F 0 "U1" H 4750 1000 60  0000 C CNN
+F 0 "U101" H 4750 1000 60  0000 C CNN
 F 1 "STM32F030C8" H 4550 2850 60  0000 C CNN
 F 2 "Housings_QFP:LQFP-48_7x7mm_Pitch0.5mm" H 4200 1950 60  0001 C CNN
@@
 	1    0    0    -1
 $EndComp
-Text Notes 6300 1200 0    60   ~ 0
-TODO: Get crystal/oscillator
 Text Notes 5100 2850 0    60   ~ 0
 TODO: Figure out comm/power header
 $Comp
-L Crystal Y1
+L Crystal Y101
 U 1 1 56529888
 P 5800 1650
-F 0 "Y1" H 5800 1800 50  0000 C CNN
+F 0 "Y101" H 5800 1800 50  0000 C CNN
 F 1 "Crystal" H 5800 1500 50  0000 C CNN
 F 2 "Crystals:Crystal_HC49-U_Vertical" H 5800 1650 60  0001 C CNN
@@
 $EndComp
 $Comp
-L C C4
+L C C102
 U 1 1 5652990D
 P 6250 1450
-F 0 "C4" H 6275 1550 50  0000 L CNN
+F 0 "C102" H 6275 1550 50  0000 L CNN
 F 1 "20P" H 6275 1350 50  0000 L CNN
 F 2 "Capacitors_SMD:C_0805" H 6288 1300 30  0001 C CNN
@@
 $EndComp
 $Comp
-L C C5
+L C C103
 U 1 1 56529966
 P 6250 1900
-F 0 "C5" H 6275 2000 50  0000 L CNN
+F 0 "C103" H 6275 2000 50  0000 L CNN
 F 1 "20P" H 6275 1800 50  0000 L CNN
 F 2 "Capacitors_SMD:C_0805" H 6288 1750 30  0001 C CNN
@@
 $EndComp
 $Comp
-L GND #PWR05
+L GND #PWR02
 U 1 1 56529BFD
 P 6800 1850
-F 0 "#PWR05" H 6800 1600 50  0001 C CNN
+F 0 "#PWR02" H 6800 1600 50  0001 C CNN
 F 1 "GND" H 6800 1700 50  0000 C CNN
 F 2 "" H 6800 1850 60  0000 C CNN
@@
 $EndComp
 Wire Wire Line
-	4700 700  4800 700
-Wire Wire Line
-	4800 700  5150 700
+	4700 700  5150 700
 Wire Wire Line
 	4700 900  4800 900
@@
 	5150 1000 5150 1100
 Wire Wire Line
-	3450 700  3850 700
-Wire Wire Line
-	3850 700  3950 700
-Wire Wire Line
-	3950 700  4100 700
+	3450 700  4100 700
 Wire Wire Line
 	3850 700  3850 900
 Wire Wire Line
-	3950 700  3950 800
-Wire Wire Line
-	3950 800  3950 900
+	3950 700  3950 900
 Connection ~ 3950 700
 Wire Wire Line
@@
 Connection ~ 3850 700
 Wire Wire Line
-	3950 3050 3950 3150
-Wire Wire Line
-	3950 3150 3950 3200
-Wire Wire Line
-	3950 3150 4050 3150
-Wire Wire Line
-	4050 3150 4700 3150
+	3950 3050 3950 3200
+Wire Wire Line
+	3950 3150 4700 3150
 Wire Wire Line
 	4050 3150 4050 3050
@@
 	2650 4550 3250 4550
 Wire Wire Line
-	5050 1450 5800 1450
-Wire Wire Line
-	5800 1450 6100 1450
+	5050 1450 6100 1450
 Wire Wire Line
 	5050 1450 5050 1600
@@
 	6400 1450 6600 1450
 Wire Wire Line
-	6600 1450 6600 1700
-Wire Wire Line
-	6600 1700 6600 1900
+	6600 1450 6600 1900
 Wire Wire Line
 	6600 1900 6400 1900
@@
 Connection ~ 6600 1700
 Wire Wire Line
-	5050 1900 5800 1900
-Wire Wire Line
-	5800 1900 6100 1900
+	5050 1900 6100 1900
 Wire Wire Line
 	5050 1900 5050 1700
@@
 BOOT0
 $Comp
-L CONN_01X10 P?
+L CONN_01X10 P102
 U 1 1 56624354
 P 1300 2050
-F 0 "P?" H 1300 2600 50  0000 C CNN
+F 0 "P102" H 1300 2600 50  0000 C CNN
 F 1 "CONN_01X10" V 1400 2050 50  0000 C CNN
-F 2 "" H 1300 2050 60  0000 C CNN
+F 2 "Pin_Headers:Pin_Header_Straight_1x10" H 1300 2050 60  0001 C CNN
 F 3 "" H 1300 2050 60  0000 C CNN
 	1    1300 2050
@@
 GPIO HEADER 1
 $Comp
-L CONN_01X04 P?
+L CONN_01X04 P105
 U 1 1 56634405
 P 5850 3900
-F 0 "P?" H 5850 4150 50  0000 C CNN
+F 0 "P105" H 5850 4150 50  0000 C CNN
 F 1 "CONN_01X04" V 5950 3900 50  0000 C CNN
-F 2 "" H 5850 3900 60  0000 C CNN
+F 2 "Pin_Headers:Pin_Header_Straight_1x04" H 5850 3900 60  0001 C CNN
 F 3 "" H 5850 3900 60  0000 C CNN
 	1    5850 3900
@@
 	6250 4050 6250 4200
 $Comp
-L GND #PWR?
+L GND #PWR03
 U 1 1 56634940
 P 6250 4200
-F 0 "#PWR?" H 6250 3950 50  0001 C CNN
+F 0 "#PWR03" H 6250 3950 50  0001 C CNN
 F 1 "GND" H 6250 4050 50  0000 C CNN
 F 2 "" H 6250 4200 60  0000 C CNN
@@
 ADC_IN8
 $Comp
-L CONN_01X04 P?
+L CONN_01X04 P103
 U 1 1 56638780
 P 5800 5200
-F 0 "P?" H 5800 5450 50  0000 C CNN
+F 0 "P103" H 5800 5450 50  0000 C CNN
 F 1 "CONN_01X04" V 5900 5200 50  0000 C CNN
-F 2 "" H 5800 5200 60  0000 C CNN
+F 2 "Pin_Headers:Pin_Header_Straight_1x04" H 5800 5200 60  0001 C CNN
 F 3 "" H 5800 5200 60  0000 C CNN
 	1    5800 5200
@@
 SPI1_NSS
 $Comp
-L CONN_01X02 P?
+L CONN_01X02 P106
 U 1 1 5663E66F
 P 7150 5300
-F 0 "P?" H 7150 5450 50  0000 C CNN
+F 0 "P106" H 7150 5450 50  0000 C CNN
 F 1 "CONN_01X02" V 7250 5300 50  0000 C CNN
-F 2 "" H 7150 5300 60  0000 C CNN
+F 2 "Pin_Headers:Pin_Header_Straight_1x02" H 7150 5300 60  0001 C CNN
 F 3 "" H 7150 5300 60  0000 C CNN
 	1    7150 5300
@@
 USART1_RX
 $Comp
-L CONN_01X10 P?
+L CONN_01X10 P101
 U 1 1 5664380D
 P 950 5100
-F 0 "P?" H 950 5650 50  0000 C CNN
+F 0 "P101" H 950 5650 50  0000 C CNN
 F 1 "CONN_01X10" V 1050 5100 50  0000 C CNN
-F 2 "" H 950 5100 60  0000 C CNN
+F 2 "Pin_Headers:Pin_Header_Straight_1x10" H 950 5100 60  0001 C CNN
 F 3 "" H 950 5100 60  0000 C CNN
 	1    950  5100
@@
 	1850 1900 1500 1900
 $Comp
-L CONN_01X02 P?
+L CONN_01X02 P104
 U 1 1 5665792F
 P 5800 7250
-F 0 "P?" H 5800 7400 50  0000 C CNN
+F 0 "P104" H 5800 7400 50  0000 C CNN
 F 1 "CONN_01X02" V 5900 7250 50  0000 C CNN
-F 2 "" H 5800 7250 60  0000 C CNN
+F 2 "Pin_Headers:Pin_Header_Straight_1x02" H 5800 7250 60  0001 C CNN
 F 3 "" H 5800 7250 60  0000 C CNN
 	1    5800 7250
@@
 Text Notes 5600 6900 0    60   ~ 0
 SENSOR I2C HEADER
+Text Notes 800  4300 0    60   ~ 0
+GPIO HEADER 2
 $EndSCHEMATC
