File: Power.sch (KiCad schematic (older format))
At the start: 22 parts, among them P301 USB_B, P302 CONN_01X02, U301 MCP1700T-3302E/TT_, U302 FT232RQ

Commit message: Ripped up previous power layout and placed all FTDI components (finished page 3 of schematic)
Connections:
- net GND: now also U302.33 (EP)
- net VCCIO: now reaches C302.1, C303.1, D302.2 (A), L301.2, R306.1, R307.1, U302.1 (VCCIO), U302.19 (VCC)
Changed lines of the file:
@@
 	-1   0    0    -1
 $EndComp
-Wire Wire Line
-	5500 1750 5500 2100
-Wire Wire Line
-	5500 1900 7200 1900
-Wire Wire Line
-	6600 1900 6600 1550
-Connection ~ 5500 1900
-Wire Wire Line
-	5500 2000 4350 2000
-Wire Wire Line
-	4350 2000 4350 1500
-Connection ~ 5500 2000
-Wire Wire Line
-	3250 950  4750 950
-Wire Wire Line
-	4350 1200 4350 950
-Wire Wire Line
-	4350 950  4400 950
-Connection ~ 4400 950
-Wire Wire Line
-	6250 950  7050 950
-Wire Wire Line
-	6600 950  6600 1250
-Connection ~ 6600 950
-Wire Wire Line
-	7200 1000 7050 1000
-Wire Wire Line
-	7050 1000 7050 950
-Wire Wire Line
-	2150 1050 2550 1050
-Wire Wire Line
-	2550 1050 2550 1600
 $Comp
 L INDUCTOR L301
@@
 	0    -1   -1   0
 $EndComp
-Wire Wire Line
-	3550 3650 4600 3650
-Wire Wire Line
-	4600 3800 4250 3800
-Wire Wire Line
-	4250 3800 4250 3650
-Connection ~ 4250 3650
-Wire Wire Line
-	1400 3500 1400 3650
-Wire Wire Line
-	1400 3650 2950 3650
 $Comp
 L C C301
@@
 	1    0    0    -1
 $EndComp
-Wire Wire Line
-	2450 4250 2450 3650
-Connection ~ 2450 3650
-Wire Wire Line
-	1100 3500 1100 4750
 $Comp
 L GND #PWR011
@@
 	1    0    0    -1
 $EndComp
-Wire Wire Line
-	900  3100 900  3750
-Wire Wire Line
-	900  3750 1100 3750
-Connection ~ 1100 3750
-Wire Wire Line
-	2450 4650 2450 4550
-Wire Wire Line
-	1100 4650 2450 4650
-Connection ~ 1100 4650
-Wire Wire Line
-	1200 3500 1200 4100
-Wire Wire Line
-	1200 4100 4600 4100
-Wire Wire Line
-	4600 3950 1300 3950
-Wire Wire Line
-	1300 3950 1300 3500
 Text HLabel 7800 3750 2    60   Input ~ 0
 TXD
@@
 	-1   0    0    1
 $EndComp
-Wire Wire Line
-	3700 2800 3700 3650
-Connection ~ 3700 3650
-Wire Wire Line
-	3700 2500 3700 950
-Connection ~ 3700 950
-Wire Wire Line
-	2950 950  2150 950
 $Comp
 L D_Schottky D302
@@
 	1    0    0    -1
 $EndComp
-Wire Wire Line
-	4000 5250 4000 3650
-Wire Wire Line
-	3350 5250 4000 5250
-Wire Wire Line
-	3700 5250 3700 5450
-Connection ~ 4000 3650
-Wire Wire Line
-	3350 5250 3350 5450
-Connection ~ 3700 5250
-Wire Wire Line
-	3700 6050 3700 5750
-Wire Wire Line
-	3350 6050 4150 6050
-Wire Wire Line
-	3350 6050 3350 5750
 $Comp
 L GND #PWR012
@@
 	1    0    0    -1
 $EndComp
-Wire Wire Line
-	3550 6150 3550 6050
-Connection ~ 3550 6050
 $Comp
 L C C304
@@
 	1    0    0    -1
 $EndComp
-Wire Wire Line
-	4600 5600 4150 5600
-Wire Wire Line
-	4150 5600 4150 5650
-Wire Wire Line
-	4150 6050 4150 5950
-Connection ~ 3700 6050
 Text GLabel 3250 5000 0    60   Input ~ 0
 NRST
-Wire Wire Line
-	3250 5000 4100 5000
 $Comp
 L R R301
@@
 	0    1    1    0
 $EndComp
-Wire Wire Line
-	4400 5000 4600 5000
 $Comp
 L GND #PWR013
@@
 	1    0    0    -1
 $EndComp
-Wire Wire Line
-	5350 6100 5350 6250
-Wire Wire Line
-	5350 6200 6000 6200
-Wire Wire Line
-	5800 6200 5800 6100
-Connection ~ 5350 6200
-Wire Wire Line
-	5650 6100 5650 6200
-Connection ~ 5650 6200
-Wire Wire Line
-	5500 6100 5500 6200
-Connection ~ 5500 6200
 $Comp
 L R R306
@@
 	0    -1   -1   0
 $EndComp
-Wire Wire Line
-	8400 4250 8400 4400
-Wire Wire Line
-	8750 4250 8750 4400
-Wire Wire Line
-	8400 4800 8400 4950
-Wire Wire Line
-	8400 4950 6550 4950
-Wire Wire Line
-	8750 4800 8750 5100
-Wire Wire Line
-	8750 5100 6550 5100
-Wire Wire Line
-	8400 3950 8400 3800
-Wire Wire Line
-	8400 3800 8750 3800
-Wire Wire Line
-	8750 3800 8750 3950
-Wire Wire Line
-	4450 3650 4450 3200
-Wire Wire Line
-	4450 3200 8600 3200
-Wire Wire Line
-	8600 3200 8600 3800
-Connection ~ 8600 3800
-Connection ~ 4450 3650
 $Comp
 L R R304
@@
 	0    1    1    0
 $EndComp
-Wire Wire Line
-	6750 4200 6550 4200
-Wire Wire Line
-	6550 4050 6750 4050
-Wire Wire Line
-	7050 4050 7300 4050
-Wire Wire Line
-	7300 4050 7300 4450
-Wire Wire Line
-	7050 4200 7300 4200
-Connection ~ 7300 4200
 $Comp
 L GND #PWR014
@@
 	1    0    0    -1
 $EndComp
-Wire Wire Line
-	6000 6200 6000 6100
-Connection ~ 5800 6200
 $Comp
 L R R302
@@
 	0    1    1    0
 $EndComp
+Text HLabel 7200 1900 2    60   Input ~ 0
+GND
+Text Label 5150 3200 0    60   ~ 0
+VCCIO
+Wire Wire Line
+	5500 1750 5500 2100
+Wire Wire Line
+	5500 1900 7200 1900
+Wire Wire Line
+	6600 1900 6600 1550
+Connection ~ 5500 1900
+Wire Wire Line
+	5500 2000 4350 2000
+Wire Wire Line
+	4350 2000 4350 1500
+Connection ~ 5500 2000
+Wire Wire Line
+	3250 950  4750 950
+Wire Wire Line
+	4350 1200 4350 950
+Wire Wire Line
+	4350 950  4400 950
+Connection ~ 4400 950
+Wire Wire Line
+	6250 950  7050 950
+Wire Wire Line
+	6600 950  6600 1250
+Connection ~ 6600 950
+Wire Wire Line
+	7200 1000 7050 1000
+Wire Wire Line
+	7050 1000 7050 950
+Wire Wire Line
+	2150 1050 2550 1050
+Wire Wire Line
+	2550 1050 2550 1600
+Wire Wire Line
+	3550 3650 4600 3650
+Wire Wire Line
+	4600 3800 4250 3800
+Wire Wire Line
+	4250 3800 4250 3650
+Connection ~ 4250 3650
+Wire Wire Line
+	1400 3500 1400 3650
+Wire Wire Line
+	1400 3650 2950 3650
+Wire Wire Line
+	2450 4250 2450 3650
+Connection ~ 2450 3650
+Wire Wire Line
+	1100 3500 1100 4750
+Wire Wire Line
+	900  3100 900  3750
+Wire Wire Line
+	900  3750 1100 3750
+Connection ~ 1100 3750
+Wire Wire Line
+	2450 4650 2450 4550
+Wire Wire Line
+	1100 4650 2450 4650
+Connection ~ 1100 4650
+Wire Wire Line
+	1200 3500 1200 4100
+Wire Wire Line
+	1200 4100 4600 4100
+Wire Wire Line
+	4600 3950 1300 3950
+Wire Wire Line
+	1300 3950 1300 3500
+Wire Wire Line
+	3700 2800 3700 3650
+Connection ~ 3700 3650
+Wire Wire Line
+	3700 2500 3700 950
+Connection ~ 3700 950
+Wire Wire Line
+	2950 950  2150 950
+Wire Wire Line
+	4000 5250 4000 3650
+Wire Wire Line
+	3350 5250 4000 5250
+Wire Wire Line
+	3700 5250 3700 5450
+Connection ~ 4000 3650
+Wire Wire Line
+	3350 5250 3350 5450
+Connection ~ 3700 5250
+Wire Wire Line
+	3700 6050 3700 5750
+Wire Wire Line
+	3350 6050 4150 6050
+Wire Wire Line
+	3350 6050 3350 5750
+Wire Wire Line
+	3550 6150 3550 6050
+Connection ~ 3550 6050
+Wire Wire Line
+	4600 5600 4150 5600
+Wire Wire Line
+	4150 5600 4150 5650
+Wire Wire Line
+	4150 6050 4150 5950
+Connection ~ 3700 6050
+Wire Wire Line
+	3250 5000 4100 5000
+Wire Wire Line
+	4400 5000 4600 5000
+Wire Wire Line
+	5350 6100 5350 6250
+Wire Wire Line
+	5350 6200 6000 6200
+Wire Wire Line
+	5800 6200 5800 6100
+Connection ~ 5350 6200
+Wire Wire Line
+	5650 6100 5650 6200
+Connection ~ 5650 6200
+Wire Wire Line
+	5500 6100 5500 6200
+Connection ~ 5500 6200
+Wire Wire Line
+	8400 4250 8400 4400
+Wire Wire Line
+	8750 4250 8750 4400
+Wire Wire Line
+	8400 4800 8400 4950
+Wire Wire Line
+	8400 4950 6550 4950
+Wire Wire Line
+	8750 4800 8750 5100
+Wire Wire Line
+	8750 5100 6550 5100
+Wire Wire Line
+	8400 3950 8400 3800
+Wire Wire Line
+	8400 3800 8750 3800
+Wire Wire Line
+	8750 3800 8750 3950
+Wire Wire Line
+	4450 3650 4450 3200
+Wire Wire Line
+	4450 3200 8600 3200
+Wire Wire Line
+	8600 3200 8600 3800
+Connection ~ 8600 3800
+Connection ~ 4450 3650
+Wire Wire Line
+	6750 4200 6550 4200
+Wire Wire Line
+	6550 4050 6750 4050
+Wire Wire Line
+	7050 4050 7300 4050
+Wire Wire Line
+	7300 4050 7300 4450
+Wire Wire Line
+	7050 4200 7300 4200
+Connection ~ 7300 4200
+Wire Wire Line
+	6000 6200 6000 6100
+Connection ~ 5800 6200
 Wire Wire Line
 	6750 3900 6550 3900
@@
 	7050 3750 7800 3750
 Connection ~ 6600 1900
-Text HLabel 7200 1900 2    60   Input ~ 0
-GND
+Wire Wire Line
+	5200 6100 5200 6150
+Wire Wire Line
+	5200 6150 5350 6150
+Connection ~ 5350 6150
 $EndSCHEMATC
