File: Hardware/CentralCommand.kicad_pcb (KiCad board)
At the start: 4 copper layers, 50.8 x 50.8 mm, 59 parts, among them P101 CONN_01X10, P102 CONN_01X10, P103 CONN_01X04, P104 CONN_01X02, P105 CONN_01X04, P106 CONN_01X02, P201 CONN_01X06, P202 CONN_01X04, P203 CONN_01X04, P204 CONN_01X03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

Commit message: Updated layout file, as that's what we're submitting to MF
Parts:
- C101, C201: value C -> MF-CAP-0805-0.1uF
- C102, C103: value 20P -> 08055A200JAT2A
- C104, C107, C301, C302, C304: value .1U -> MF-CAP-0805-0.1uF
- C105, C108: value 1U -> MCSH31B105K100CT
- C106, C109: value 10U -> MC1206B106K160CT
- C303: value 4.7U -> GRM32RR71C475KA01L
- C305, C306: value 10U -> MF-CAP-1206-10uF
- D301, D302: value D_Schottky -> B130-13-F
- D303, D304: value LED -> SML-LXT0805GW-TR
- L101: value INDUCTOR -> LQH31CN100K03L
- L301: value FERRITE -> 742792605
- P202, P203: value CONN_01X04 -> CONN_01X04_2mm
- P301: value USB_B -> 10118193
- R201, R202, R204: value R -> MF-RES-0805-10K
- R203, R206, R207, R208, R209, R301, R302, R303: value 0 -> MF-RES-0805-0
- R306, R307: value 270 -> MCWR08X2700FTL
- SW201: value FSM2JSMAA-ND -> FSM2JSMAA
- U101: value STM32F030C8 -> STM32F030C8T6
- U302: value FT232RQ -> FT232RQ-REEL
- Y101: value Crystal -> FOXSLF/080-20
Connections:
- P301 pad 6: GND -> (no net)
- P301 pad 7: GND -> (no net)
- P301 pad 8: GND -> (no net)
- P301 pad 9: GND -> (no net)
